Commit message: NO_05

File: my_robo_description/my_robo.urdf (robot description, URDF)
Before this commit: robot my_robo, 5 links, 4 joints
Links:
- added link pico_flexx_depth_frame
- added link pico_flexx_link, mass 1; collision box size=0.007 0.066 0.016; visual box size=0.007 0.066 0.016
- added link pico_flexx_link_optical_frame
Joints:
- added joint pico_flexx_base_joint: type fixed, parent base_link, child pico_flexx_link_optical_frame, origin xyz=0.2 0 0.07 rpy=0 0 0
- added joint pico_flexx_depth_joint: type fixed, parent pico_flexx_link_optical_frame, child pico_flexx_depth_frame, origin xyz=0 0 0 rpy=${-M_PI/2} 0 ${-M_PI/2}
- added joint pico_flexx_joint: type fixed, parent pico_flexx_link_optical_frame, child pico_flexx_link, origin xyz=0 0 0 rpy=0 0 0

Commit message: for NO_06

File: my_robo_description/my_robo.urdf (robot description, URDF)
Before this commit: robot my_robo, 8 links, 7 joints
Links:
- removed link pico_flexx_depth_frame
- removed link pico_flexx_link
- removed link pico_flexx_link_optical_frame
- added link hokuyo_link, mass 1e-5; collision box size=0.1 0.1 0.1; visual mesh filename=package://rrbot_description/meshes/hokuyo.dae
Joints:
- removed joint pico_flexx_base_joint
- removed joint pico_flexx_depth_joint
- removed joint pico_flexx_joint
- added joint hokuyo_joint: type fixed, parent base_link, child hokuyo_link, origin xyz=0.2 0 0.07 rpy=0 0 0, axis 0 1 0
